File: _autosave-Pheripheral-Scout.kicad_sch (KiCad schematic)
At the start: 6 parts

Commit message: First
Parts:
- removed J? (x4): B2B-XH-A_LF__SN_, digikey-footprints:PinHeader_1x2_P2.5mm_Drill1.1mm, symbol dk_Rectangular-Connectors-Headers-Male-Pins:B2B-XH-A_LF__SN_
- removed J?: B4B-XH-A_LF__SN_, digikey-footprints:PinHeader_1x4_P2.5mm_Drill1.1mm, symbol dk_Rectangular-Connectors-Headers-Male-Pins:B4B-XH-A_LF__SN_
- removed J?: Conn_02x07_Top_Bottom, Connector_IDC:IDC-Header_2x07_P2.54mm_Vertical, symbol Connector_Generic:Conn_02x07_Top_Bottom
- added J?: Conn_02x07_Top_Bottom, Connector_IDC:IDC-Header_2x07_P2.54mm_Vertical, symbol Connector_Generic:Conn_02x07_Top_Bottom
- added J?: Bottom_Lights, digikey-footprints:PinHeader_1x2_P2.5mm_Drill1.1mm, symbol dk_Rectangular-Connectors-Headers-Male-Pins:B2B-XH-A_LF__SN_
- added J?: Switch_2, digikey-footprints:PinHeader_1x2_P2.5mm_Drill1.1mm, symbol dk_Rectangular-Connectors-Headers-Male-Pins:B2B-XH-A_LF__SN_
- added J?: Motor, digikey-footprints:PinHeader_1x4_P2.5mm_Drill1.1mm, symbol dk_Rectangular-Connectors-Headers-Male-Pins:B4B-XH-A_LF__SN_
- added J?: Switch_1, digikey-footprints:PinHeader_1x2_P2.5mm_Drill1.1mm, symbol dk_Rectangular-Connectors-Headers-Male-Pins:B2B-XH-A_LF__SN_
- added J?: Top_Lights, digikey-footprints:PinHeader_1x2_P2.5mm_Drill1.1mm, symbol dk_Rectangular-Connectors-Headers-Male-Pins:B2B-XH-A_LF__SN_
