File: Pheripheral-Scout.kicad_sch (KiCad schematic)
At the start: 6 parts

Commit message: Alpha Prototype ready
Parts:
- J1, J2, J3, J4: renamed from J?; footprint digikey-footprints:PinHeader_1x2_P2.5mm_Drill1.1mm -> digikey-footprints:PinHeader_1x2_P2mm_Drill1mm; Description_1 (none) -> CONN HEADER VERT 2POS 2.5MM
- J5: renamed from J?; footprint digikey-footprints:PinHeader_1x4_P2.5mm_Drill1.1mm -> digikey-footprints:PinHeader_1x4_P2mm_Drill1mm; Description_1 (none) -> CONN HEADER VERT 4POS 2.5MM
- gave numbers to parts that had none: 1
Connections:
- net 1A: now also J5.3; no longer J5.1A
- net 1B: now also J5.4; no longer J5.1B
- net 2A: now also J5.2; no longer J5.2A
- net 2B: now also J5.1; no longer J5.2B
- net BL_Anode: now also J2.2; no longer J2.+
- net BL_Cathode: now also J2.1; no longer J2.-
- net TL_Anode: now also J1.2; no longer J1.+
- net TL_Cathode: now also J1.1; no longer J1.-
- net GND: now reaches J6.13 (Pin_13)
- net GND: now also J6.14 (Pin_14)
Other:
- moved on the sheet: J1, J2, J3, J4, J5

Commit message: Updated BOM
Parts:
- J6: value Conn_02x07_Top_Bottom -> CA2314PA10Z
Changed lines of the file:
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@@
 			)
 		)
-		(property "Value" "Conn_02x07_Top_Bottom"
+		(property "Value" "CA2314PA10Z"
 			(at 123.19 63.5 0)
 			(effects
@@
 			)
 		)
-		(property "Datasheet" "~"
+		(property "Datasheet" "https://mm.digikey.com/Volume0/opasdata/d220001/medias/docus/2689/CA2305SA.pdf"
 			(at 121.92 74.93 0)
 			(effects
@@
 			)
 		)
-		(property "Description" ""
+		(property "Description" "https://www.digikey.com/en/products/detail/cvilux-usa/CA2314PA10Z/15519144"
 			(at 121.92 74.93 0)
 			(effects
